File: kicad/ferro-dactyl.sch (KiCad schematic (older format))
At the start: 65 parts

Commit message: Adds pcb
Parts:
- removed D? (x32): 1N4148, Diode_THT:D_DO-35_SOD27_P7.62mm_Horizontal, symbol Diode:1N4148
- removed SW? (x32): SW_Push, symbol Switch:SW_Push
- added D1, D2, D3, D4, D5: LED, Connector_PinSocket_2.54mm:PinSocket_1x02_P2.54mm_Vertical, symbol Device:LED
- added J1: Columns, Connector_PinSocket_2.54mm:PinSocket_1x06_P2.54mm_Vertical, symbol Connector_Generic:Conn_01x06
- added J2: Rows, Connector_PinSocket_2.54mm:PinSocket_1x06_P2.54mm_Vertical, symbol Connector_Generic:Conn_01x06
- added J3: UART, Connector_PinSocket_2.54mm:PinSocket_1x04_P2.54mm_Vertical, symbol Connector_Generic:Conn_01x04
- added J4: SSD 1306, Connector_PinSocket_2.54mm:PinSocket_1x04_P2.54mm_Vertical, symbol Connector_Generic:Conn_01x04
- added JP1: Left/Right, Connector_PinHeader_2.54mm:PinHeader_1x03_P2.54mm_Vertical, symbol Jumper:Jumper_3_Open
- added Q1: BC547, Package_TO_SOT_THT:TO-92_Inline, symbol Transistor_BJT:BC547
- added R1: 330, Resistor_THT:R_Axial_DIN0411_L9.9mm_D3.6mm_P12.70mm_Horizontal, symbol Device:R
- added R2, R3, R4, R5, R6: 180, Resistor_THT:R_Axial_DIN0411_L9.9mm_D3.6mm_P12.70mm_Horizontal, symbol Device:R
- BP?1: renamed from BP??; footprint (none) -> YAAJ_STM32:YAAJ_BluePill_SWD_1
Connections:
- net SCL: now reaches BP?1.14 (PB6)
- net SCL: now also J4.2 (Pin_2)
- net SDA: now reaches BP?1.15 (PB7)
- net SDA: now also J4.1 (Pin_1)
- net LED: now reaches BP?1.16 (PB8)
- net LED: now also R1.2
- net LR: now reaches BP?1.17 (PB9)
- net LR: now also JP1.2 (C)
- net +5V: now reaches BP?1.18 (5V)
- net +5V: now also J3.1 (Pin_1), R2.1, R3.1, R4.1, R5.1, R6.1
- net GND: now reaches BP?1.19 (GND)
- net GND: now also BP?1.39 (GND), BP?1.40 (GND), J3.4 (Pin_4), J4.4 (Pin_4), JP1.3 (B), Q1.3 (E)
- net +3V3: now reaches BP?1.20 (3V3)
- net +3V3: now also J4.3 (Pin_3), JP1.1 (A)
- net COL6: now reaches BP?1.25 (PA0)
- net COL6: now also J1.6 (Pin_6)
- net COL5: now reaches BP?1.26 (PA1)
- net COL5: now also J1.5 (Pin_5)
- net COL4: now reaches BP?1.27 (PA2)
- net COL4: now also J1.4 (Pin_4)
- net COL3: now reaches BP?1.28 (PA3)
- net COL3: now also J1.3 (Pin_3)
- net COL2: now reaches BP?1.29 (PA4)
- net COL2: now also J1.2 (Pin_2)
- net COL1: now reaches BP?1.30 (PA5)
- net COL1: now also J1.1 (Pin_1)
- net ROW6: now reaches BP?1.31 (PA6)
- net ROW6: now also J2.6 (Pin_6)
- net ROW5: now reaches BP?1.32 (PA7)
- net ROW5: now also J2.5 (Pin_5)
- net ROW4: now reaches BP?1.33 (PB0)
- net ROW4: now also J2.4 (Pin_4)
- net ROW3: now reaches BP?1.34 (PB1)
- net ROW3: now also J2.3 (Pin_3)
- net ROW2: now reaches BP?1.35 (PB10)
- net ROW2: now also J2.2 (Pin_2)
- net ROW1: now reaches BP?1.36 (PB11)
- net ROW1: now also J2.1 (Pin_1)
- net TX: now reaches BP?1.6 (PA9)
- net TX: now also J3.2 (Pin_2)
- net RX: now reaches BP?1.7 (PA10)
- net RX: now also J3.3 (Pin_3)
- new net: D1.1 (K), D2.1 (K), D3.1 (K), D4.1 (K), D5.1 (K), Q1.1 (C)
- new net: D1.2 (A), R2.2
- new net: Q1.2 (B), R1.1
- new net: D2.2 (A), R3.2
- new net: D3.2 (A), R4.2
- new net: D4.2 (A), R5.2
- new net: D5.2 (A), R6.2
- no-connect marks 0 -> 17
Other:
- moved on the sheet: BP?1
